Commit message: feat: YAML robot spec loader — define custom robots or humanoid variants without URDF (14 tests)

File: examples/robots/rrbot.urdf (robot description, URDF)
Before this commit: robot rrbot, 3 links, 2 joints
Links:
- added link tool0; visual box size=0.08 0.06 0.06
Joints:
- added joint tool0_fixed: type fixed, parent link2, child tool0, origin xyz=0.50 0 0 rpy=0 0 0
